Commit message: renders + lidar sensor description

File: urdf/Robot_description/urdf/Robot.xacro (robot description, xacro)
@@ -4,5 +4,5 @@
 <xacro:include filename="$(find Robot_description)/urdf/Robot.trans" />
 <xacro:include filename="$(find Robot_description)/urdf/Robot.gazebo" />
-<link name="base_link">
+<!-- <link name="base_link">
   <inertial>
     <origin rpy="0 0 0" xyz="0.27548548877366963 0.1607766931435237 0.7499221587595302"/>
@@ -76,3 +76,104 @@
   <axis xyz="1.0 0.0 -0.0"/>
 </joint>
+ -->
+<link name="base_link">
+  <inertial>
+    <origin rpy="0 0 0" xyz="0 0 0"/>
+    <mass value="2812.7218319396366"/>
+    <inertia ixx="709.712889" ixy="-0.002526" ixz="-0.001489" iyy="749.567607" iyz="13.56912" izz="142.476075"/>
+  </inertial>
+  <visual>
+    <origin rpy="0 0 0" xyz="0 0 0"/>
+    <geometry>
+      <mesh filename="package://Robot_description/meshes/base_link.stl" scale="0.001 0.001 0.001"/>
+    </geometry>
+    <material name="silver"/>
+  </visual>
+  <collision>
+    <origin rpy="0 0 0" xyz="0 0 0"/>
+    <geometry>
+      <mesh filename="package://Robot_description/meshes/base_link.stl" scale="0.001 0.001 0.001"/>
+    </geometry>
+  </collision>
+</link>
+<link name="wheel_l_1">
+  <inertial>
+    <origin rpy="0 0 0" xyz="0 0 0"/>
+    <mass value="120.84136142033135"/>
+    <inertia ixx="2.370587" ixy="0.0" ixz="0.0" iyy="1.343134" iyz="-0.0" izz="1.343134"/>
+  </inertial>
+  <visual>
+    <origin rpy="0 0 0" xyz="-0 -0 -0"/>
+    <geometry>
+      <mesh filename="package://Robot_description/meshes/wheel_l_1.stl" scale="0.001 0.001 0.001"/>
+    </geometry>
+    <material name="silver"/>
+  </visual>
+  <collision>
+    <origin rpy="0 0 0" xyz="-0 -0 -0"/>
+    <geometry>
+      <mesh filename="package://Robot_description/meshes/wheel_l_1.stl" scale="0.001 0.001 0.001"/>
+    </geometry>
+  </collision>
+</link>
+<link name="wheel_r_1">
+  <inertial>
+    <origin rpy="0 0 0" xyz="-0 -0 -0"/>
+    <mass value="120.84136142033135"/>
+    <inertia ixx="2.370587" ixy="0.0" ixz="0.0" iyy="1.343134" iyz="0.0" izz="1.343134"/>
+  </inertial>
+  <visual>
+    <origin rpy="0 0 0" xyz="-0 -0 -0"/>
+    <geometry>
+      <mesh filename="package://Robot_description/meshes/wheel_r_1.stl" scale="0.001 0.001 0.001"/>
+    </geometry>
+    <material name="silver"/>
+  </visual>
+  <collision>
+    <origin rpy="0 0 0" xyz="-0 -0 -0"/>
+    <geometry>
+      <mesh filename="package://Robot_description/meshes/wheel_r_1.stl" scale="0.001 0.001 0.001"/>
+    </geometry>
+  </collision>
+</link>
+<joint name="Rev3" type="continuous">
+  <origin rpy="0 0 0" xyz="0.35 -0.2 0.15"/>
+  <parent link="base_link"/>
+  <child link="wheel_l_1"/>
+  <axis xyz="-1.0 0.0 0.0"/>
+</joint>
+<!--  Falta ver el offset de ruedas -->
+<joint name="Rev4" type="continuous">
+  <origin rpy="0 0 0" xyz="-0.35 -0.2 0.15"/>
+  <parent link="base_link"/>
+  <child link="wheel_r_1"/>
+  <axis xyz="1.0 0.0 -0.0"/>
+</joint>
+<!-- Sensor description -->
+<!-- Hokuyo Laser1 -->
+  <link name="laser1_link">
+    <collision>
+      <origin xyz="0 0 0" rpy="0 0 0"/>
+      <geometry>
+         <box size="0.005 0.005 0.005"/>
+      </geometry>
+    </collision>
+    <visual>
+      <origin xyz="0 0 0" rpy="0 0 0"/>
+      <geometry>
+         <box size="0.005 0.005 0.005"/>
+      </geometry>
+    </visual>
+    <inertial>
+      <mass value="1e-5" />
+      <origin xyz="0 0 0" rpy="0 0 0"/>
+      <inertia ixx="1e-6" ixy="0" ixz="0" iyy="1e-6" iyz="0" izz="1e-6" />
+    </inertial>
+  </link>
+  <joint name="laser1_joint" type="fixed">
+    <axis xyz="0 1 0" />
+    <origin xyz="0.06 -0.03 0" rpy="0 0 0"/>
+    <parent link="base"/>
+    <child link="laser1_link"/>
+  </joint>
 </robot>
